File: schematics/TableBoard/ButtonBoard.kicad_sch (KiCad schematic)
At the start: 1 part, among them J4 Conn_01x06_Male

Commit message: v2 schematics
Connections:
- net +5V: now also J4.2 (Pin_2); no longer J4.1 (Pin_1)
- net GND: now also J4.1 (Pin_1); no longer J4.2 (Pin_2)
Changed lines of the file:
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@@
 (kicad_sch (version 20211123) (generator eeschema)
   (paper "A4")
-  (wire (pts (xy 173.99 91.44) (xy 187.96 91.44))
+  (wire (pts (xy 173.99 88.9) (xy 194.31 88.9))
     (stroke (width 0) (type default) (color 0 0 0 0))
   )
-  (wire (pts (xy 173.99 88.9) (xy 187.96 88.9))
+  (wire (pts (xy 173.99 91.44) (xy 187.96 91.44))
     (stroke (width 0) (type default) (color 0 0 0 0))
   )
@@
     (pin "6")
   )
-  (symbol (lib_id "power:+5V") (at 187.96 88.9 0) (unit 1)
+  (symbol (lib_id "power:+5V") (at 187.96 91.44 0) (unit 1)
     (in_bom yes) (on_board yes) (fields_autoplaced)
-    (property "Reference" "#PWR013" (id 0) (at 187.96 92.71 0)
+    (property "Reference" "#PWR013" (id 0) (at 187.96 95.25 0)
       (effects (font (size 1.27 1.27)) hide)
     )
-    (property "Value" "+5V" (id 1) (at 187.96 83.82 0))
-    (property "Footprint" "" (id 2) (at 187.96 88.9 0)
-      (effects (font (size 1.27 1.27)) hide)
-    )
-    (property "Datasheet" "" (id 3) (at 187.96 88.9 0)
-      (effects (font (size 1.27 1.27)) hide)
-    )
-    (pin "1")
-  )
-  (symbol (lib_id "power:GND") (at 187.96 91.44 0) (unit 1)
-    (in_bom yes) (on_board yes) (fields_autoplaced)
-    (property "Reference" "#PWR014" (id 0) (at 187.96 97.79 0)
-      (effects (font (size 1.27 1.27)) hide)
-    )
-    (property "Value" "GND" (id 1) (at 187.96 96.52 0))
+    (property "Value" "+5V" (id 1) (at 187.96 86.36 0))
     (property "Footprint" "" (id 2) (at 187.96 91.44 0)
       (effects (font (size 1.27 1.27)) hide)
@@
       (effects (font (size 1.27 1.27)) hide)
     )
+    (pin "1")
+  )
+  (symbol (lib_id "power:GND") (at 194.31 88.9 0) (unit 1)
+    (in_bom yes) (on_board yes) (fields_autoplaced)
+    (property "Reference" "#PWR014" (id 0) (at 194.31 95.25 0)
+      (effects (font (size 1.27 1.27)) hide)
+    )
+    (property "Value" "GND" (id 1) (at 194.31 93.98 0))
+    (property "Footprint" "" (id 2) (at 194.31 88.9 0)
+      (effects (font (size 1.27 1.27)) hide)
+    )
+    (property "Datasheet" "" (id 3) (at 194.31 88.9 0)
+      (effects (font (size 1.27 1.27)) hide)
+    )
