File: schematics/TableBoard/TableBoard.kicad_pcb (KiCad board)
At the start: 2 copper layers, 101.6 x 66 mm, 14 parts, among them J1 Barrel_Jack_MountingPin, J2 Conn_01x04_Male, J3 Conn_01x04_Male, J4 Conn_01x06_Male, J5 Conn_01x06_Female, J6 Conn_01x06_Female

Commit message: v2 schematics
Parts:
- A1, A2, A3, J2, J3, J4, J5, J6: moved to B.Cu
- moved J4 71.1 mm to (92.7, 73.7)
- moved A2 57.5 mm to (27.9, 33.0), turned to -90 degrees
- moved J2 50.7 mm to (45.7, 23.9), turned to 180 degrees
- moved C1 30.7 mm to (52.1, 35.6), turned to -90 degrees
- moved J6 22.9 mm to (88.9, 34.3)
- moved J5 22.7 mm to (101.6, 52.1)
- moved A3 18.0 mm to (58.4, 33.0), turned to -90 degrees
- moved C2 14.5 mm to (82.5, 36.8), turned to -90 degrees
- moved J3 10.5 mm to (74.9, 23.9), turned to 180 degrees
- moved A1 9.14 mm to (43.2, 55.9), turned to -90 degrees
Connections:
- J4 pad 1: +5V -> GND
- J4 pad 2: GND -> +5V
Routing:
- net GND: track 247.6 -> 11.1 mm
- net +5V: track 147.7 -> 169.1 mm
- net /LeftMotor/DIR: track 22.7 -> 30.4 mm
- net /ButtonBoard/LeftUp: track 25.0 -> 32.0 mm
- net /LeftMotor/STEP: track 22.7 -> 29.6 mm
- net /LeftMotor/NENABLE: track 33.1 -> 38.7 mm
- net /ButtonBoard/RightUp: track 25.0 -> 21.2 mm
- net /ButtonBoard/Up: track 25.0 -> 28.4 mm
- net +12V: track 102.9 -> 104.8 mm
- net /RightMotor/C: track 9.02 -> 10.7 mm
- net /RightMotor/B: track 9.04 -> 10.7 mm
- net /RightMotor/A: track 9.05 -> 10.7 mm
- net /RightMotor/D: track 9.03 -> 10.7 mm
- net /RightMotor/STEP: track 10.2 -> 11.2 mm
- net /RightMotor/DIR: track 10.2 -> 11.2 mm
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